File: hardware/Nixie-Uhr/Nixie-Treiber-IN12b-V1_2.brd (EAGLE design)
At the start: 158.5 x 80 mm, 88 parts, among them IC1 74141N, IC10 MC34063, IC11 DS1307, IC12 LM2574, IC13 LD1117, IC14 ESP07, IC2 74141N, IC3 74141N, IC4 74141N, IC5 74141N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

Commit message: Hardware description updated.
Parts:
- C10.1: value 1000uF/35V -> 1000uF
- C10.5: value 10uF/250V -> 22µF/400V
- D10.1: value BYV26 -> BA157
- L10.1: value 330uH -> 390uH
- T10.2: value SPP20N60 -> IRFB812PBF
- moved Q1 0.12 mm to (97.8, 39.3), flipped to the top
- renumbered Q2 to T10.3, R1 to R10.7, R2 to R10.6
Connections:
- net N$39 renamed TX1
Routing:
- net VIN: track 11.9 -> 0.00 mm
- net N$26: track 3.45 -> 8.06 mm, vias 0 -> 1
- net N$25: track 6.02 -> 5.52 mm, vias 0 -> 1
Other:
- board text added: "12V / 500mA"
- board text added: "35V"
- board text added: "3V3"
- board text added: "5V"
- board text added: "ADC"
- board text added: "DTR"
- board text added: "GPIO12"
- board text added: "GPIO14"
- board text added: "GPIO16"
- board text added: "HV"
- board text added: "HV-Einstellung"
- board text added: "Minuten-E"
- board text added: "Minuten-Z"
- board text added: "Nixie-Treiber 1.2"
- board text added: "Nixie-Treiber 1.2 NTP-Time Server"
- board text added: "Port-Anschluss auch als Buchse"
- board text added: "RTS"
- board text added: "RX"
- board text added: "Sekunden-E"
- board text added: "Sekunden-Z"
- board text added: "Stunden-E"
- board text added: "Stunden-Z"
- board text added: "TX"
- board text added: "Test- Masse"
- board text added: "USB-Ser.-Anschluss"
- board text added: "u. Punkte"
- board text removed: "Nixie-Treiber 1.0"
- board text removed: "Nixie-Treiber 1.0 NTP-Time Server"
