File: hardware/Nixie-Uhr/Nixie-Treiber-IN12b-V1_2.sch (EAGLE design)
At the start: 88 parts, among them IC1 74141N, IC10 MC34063, IC11 DS1307, IC12 LM2574, IC13 LD1117, IC14 ESP07, IC2 74141N, IC3 74141N, IC4 74141N, IC5 74141N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

Commit message: Hardware description updated.
Parts:
- C10.1: value 1000uF/35V -> 1000uF
- C10.5: value 10uF/250V -> 22µF/400V
- D10.1: value BYV26 -> BA157
- L10.1: value 330uH -> 390uH
- T10.2: value SPP20N60 -> IRFB812PBF
- renumbered Q2 to T10.3, R1 to R10.7, R2 to R10.6
Connections:
- net N$39 renamed TX1
Other:
- note added: "Anodenspanung ca. 180V"
- note added: "I2C-Adapter 3V3"
- note added: "I2C-Adapter 5V"
- note added: "Port-Stecker für GPIO 5 und 3V3 Versorgung"
- note added: "Stecker vorbereitet für FT232-3V3 USB-Serial Adapter"
- note removed: "'Highest Expander'"
- note removed: "'MY_SCL'"
- note removed: "'MY_SDA'"
- note removed: "'Power Control'"
- note removed: "<= 500 mA"
- note removed: "Level Converter"
- note removed: "Lithiumbatterie"
- note removed: "Oberere Punkte (Dot Control)"
- note removed: "PIN 13 und 14 sind beim ESP8266-07 vertauscht!"
- note removed: "Reset Generator"
- note removed: "Unterere Punkte (Dot Control)"
- note removed: "max. 200 Volt"
- moved on the sheet: IC13, IC3, IC4, IC5, IC6, IC7, IC8, R14.11, SV1, SV3, SV4, SV5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
